File: Turn signals/Turn signals.kicad_sch (KiCad schematic)
At the start: 23 parts, among them J1 Conn_SW, J2 Conn_FWD_L, J3 Conn_BWD_L, J4 Conn_FWD_R, J5 Conn_BWD_R, J6 Conn_SW, Q1 IRLZ44N, U1 ICM7555, U2 MT3608

Commit message: 2024-04-11
Parts:
- removed BT1: CR2032, Custom:BatteryHolder_multicomp_CH28-2032LF, symbol Device:Battery_Cell
- removed C3, C4: 22uF, Custom:0603_1608Metric_Pad_HandSolder_Valuea, symbol Device:C
- removed D2: B230, Diode_SMD:D_SMB, symbol Diode:B230
- removed J1: Conn_SW, symbol Connector_Generic:Conn_01x05
- removed J2: Conn_FWD_L, Connector_Molex:Molex_KK-254_AE-6410-02A_1x02_P2.54mm_Vertical, symbol Connector_Generic:Conn_01x02
- removed J3: Conn_BWD_L, Connector_Molex:Molex_KK-254_AE-6410-02A_1x02_P2.54mm_Vertical, symbol Connector_Generic:Conn_01x02
- removed J4: Conn_FWD_R, Connector_Molex:Molex_KK-254_AE-6410-02A_1x02_P2.54mm_Vertical, symbol Connector_Generic:Conn_01x02
- removed J5: Conn_BWD_R, Connector_Molex:Molex_KK-254_AE-6410-02A_1x02_P2.54mm_Vertical, symbol Connector_Generic:Conn_01x02
- removed J6: Conn_SW, Connector_Molex:Molex_KK-254_AE-6410-05A_1x05_P2.54mm_Vertical, symbol Connector_Generic:Conn_01x05
- removed L1: 4.7uH, Inductor_SMD:L_Bourns_SRP7028A_7.3x6.6mm, symbol Device:L
- removed R3: 715, Custom:0603_1608Metric_Pad_HandSolder_Valuea, symbol Device:R
- removed R4: 115, Custom:0603_1608Metric_Pad_HandSolder_Valuea, symbol Device:R
- removed R5: 0, Resistor_SMD:R_0603_1608Metric_Pad0.98x0.95mm_HandSolder, symbol Device:R
- removed R6: R, Custom:0603_1608Metric_Pad_HandSolder_Valuea, symbol Device:R
- removed U2: MT3608, Package_TO_SOT_SMD:SOT-23-6, symbol Regulator_Switching:MT3608
- added D1, D2, D3, D4, D5, D6, D7, D8: LED, symbol Device:LED
- C1: value C -> 2.2uF; symbol Device:C -> Device:C_Polarized
- Q1: value IRLZ44N -> C2383; symbol Transistor_FET:IRLZ44N -> Device:Q_NPN_ECB
- R1: value 100K -> 4.7K
- R2: value R -> 200K
- R7: value R -> 4.7K
Connections:
- net LED_R is gone; now on net P: S1.3 (4)
- net GND: now also Q1.1 (E); no longer Q1.3 (S), R1.1
- net VCC: now also S1.2 (3); no longer U1.8 (VCC)
- net at R7.2: now also Q1.3 (B); no longer Q1.1 (G)
- net A: now reaches C1.1, R2.1, U1.2 (TRIG), U1.6 (THR)
- net at Q1.2 (C): now also R1.1
- net +3V0: no longer names the net of S1.5 (7)
- net +3V0: now also R1.2; no longer S1.2 (3)
- removed net EN_OUT: R1.2, S1.4 (5), S1.6 (8), U1.4 (RESET)
- net LED_L renamed P
- net P: now also U1.4 (RESET), U1.8 (VCC), D2.2 (A), D4.2 (A), D6.2 (A), D8.2 (A)
- new net: D1.2 (A), D2.1 (K)
- new net: D5.2 (A), D6.1 (K)
- new net: D3.2 (A), D4.1 (K)
- new net: D7.2 (A), D8.1 (K)
- new net L: D1.1 (K), D3.1 (K), S1.4 (5)
- new net R: D5.1 (K), D7.1 (K), S1.6 (8)
Other:
- note removed: "Astable 555"
- note removed: "DC Step-up (optional)"
- note removed: "Switch (not on board)"
- moved on the sheet: R2, R7, S1
