File: LED driver/bms.kicad_sch (KiCad schematic)
At the start: 0 parts

Commit message: 2024-04-17
Changed lines of the file:
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@@
-		)
-	)
-	(hierarchical_label "C-"
-		(shape input)
-		(at 107.95 120.65 0)
-		(fields_autoplaced yes)
-		(effects
-			(font
-				(size 1.27 1.27)
-			)
-			(justify left)
 		)
 	)
