File: LED driver/LED remote.kicad_sch (KiCad schematic)
At the start: 48 parts, among them J1 Conn_UART, J2 USB_C_Receptacle_USB2.0_14P, SW1 EN, SW10 SW_Push, SW2 ON/OFF, SW3 MENU, SW4 LEFT, SW5 UP, SW6 OK, SW7 DOWN, SW8 BACK, SW9 RIGHT, U1 TPS63001, U2 ADXL343, U3 74HC165, U4 ESP32-C3-MINI-1-N4

Commit message: 2024-04-17
Parts:
- removed BT2: 2x AAA, symbol Device:Battery
- removed J1: Conn_UART, Connector_PinHeader_2.54mm:PinHeader_1x04_P2.54mm_Vertical, symbol Connector_Generic:Conn_01x04
- removed J2: USB_C_Receptacle_USB2.0_14P, symbol Connector:USB_C_Receptacle_USB2.0_14P
- removed JP3: SolderJumper_2_Open, Jumper:SolderJumper-2_P1.3mm_Open_RoundedPad1.0x1.5mm, symbol Jumper:SolderJumper_2_Open
- removed R10, R9: 100K, symbol Device:R
- removed R14, R15: 0, Resistor_SMD:R_0603_1608Metric_Pad0.98x0.95mm_HandSolder, symbol Device:R_Small
- added C5, C6: 1uF, symbol Device:C
- added D1: MP001251, Custom:LED_MP001251_3.5x2.8mm, symbol Device:LED_RGB
- added J1: USB4105-GF-A, Connector_USB:USB_C_Receptacle_GCT_USB4105-xx-A_16P_TopMnt_Horizontal, symbol Connector:USB_C_Receptacle_USB2.0_14P
- added J2: Conn_UART, Connector_PinHeader_1.00mm:PinHeader_1x03_P1.00mm_Vertical_SMD_Pin1Left, symbol Connector:Conn_01x03_Socket
- added R12, R13, R14: 4.7K, symbol Device:R
- added R7: 5.1K, symbol Device:R
- added RN1: YC248-JR-074K7L, footprints:RES_YC248_4X1P6_YAG, symbol Device:R_Network08
- added U2: MCP73833-AMI/UN, Package_SO:MSOP-10_3x3mm_P0.5mm, symbol Battery_Management:MCP73833-xxx-UN
- BT1: footprint (none) -> footprints:S2BPHSM4TBLFSN; now fitted
- JP1: footprint (none) -> Jumper:SolderJumper-2_P1.3mm_Open_RoundedPad1.0x1.5mm
- L1: value L -> 2.2uH
- R10: renamed from R12; value 100K -> 10K
- R11: renamed from R13; value 100K -> 10K
- R15: renamed from R7; value 100K -> ~24K
- R2, R3: value 100K -> 100
- R4: value 100K -> 150
- R5: value 100K -> 1K
- R6: value 100K -> 10K
- R8: value 100K -> 5.1K
- SW1: value EN -> JS102000SAQN; footprint (none) -> Custom:SW_SPDT_CK_JS102011SAQN
- SW10: renamed from SW9; footprint (none) -> Button_Switch_THT:SW_PUSH_6mm_H4.3mm
- SW3: renamed from SW2; footprint (none) -> Button_Switch_THT:SW_PUSH_6mm_H4.3mm
- SW4: renamed from SW3; footprint (none) -> Button_Switch_THT:SW_PUSH_6mm_H4.3mm
- SW5: renamed from SW4; footprint (none) -> Button_Switch_THT:SW_PUSH_6mm_H4.3mm
- SW6: renamed from SW5; footprint (none) -> Button_Switch_THT:SW_PUSH_6mm_H4.3mm
- SW7: renamed from SW6; footprint (none) -> Button_Switch_THT:SW_PUSH_6mm_H4.3mm
- SW8: renamed from SW7; footprint (none) -> Button_Switch_THT:SW_PUSH_6mm_H4.3mm
- SW9: renamed from SW8; footprint (none) -> Button_Switch_THT:SW_PUSH_6mm_H4.3mm
- U3: renamed from U4; footprint ESP32C3MINI1N4 -> ESP32-C3-MINI-1-N4:ESP32C3MINI1N4
- U4: renamed from U3; value 74HC165 -> MC74HC165ADG; footprint (none) -> Package_SO:SOIC-16_3.9x9.9mm_P1.27mm
- U5: renamed from U2; value ADXL343 -> ADXL345BCCZ
- renumbered C7 to C10, C6 to C11, C5 to C12, C9 to C7, C10 to C9, R11 to R9, SW10 to SW2
Connections:
- net +3.3V is gone; now on net +3V3: C8.2, C9.2, R10.1, R11.1, R9.1, U3.3 (3V3)
- net BMS/O+ is gone; now on net V_{BAT}: C1.1, R1.1, U1.5 (VIN)
- net BMS/O- is gone; now on net GND: JP1.2 (B), SW1.2 (B)
- net IO0 is gone; now on net SCL: U3.12 (IO0)
- net IO1 is gone; now on net SDA: U3.13 (IO1)
- net IO3 is gone; now on net Q7: U3.6 (IO3)
- net IO4 is gone; now on net CP: U3.18 (IO4)
- net IO5 is gone; now on net SH/~{LD}: U3.19 (IO5)
- net IO6 is gone; now on net INT1: U3.20 (IO6)
- net IO7 is gone; now on net INT2: U3.21 (IO7)
- net +3V3: now also R12.2, R13.2, R14.2; no longer U5.12 (SDO/ADDR)
- net GND: now also C5.2, C6.2, J1.A1 (GND), J1.A12 (GND), J1.B1 (GND), J1.B12 (GND), J1.S1 (SHIELD), J2.1 (Pin_1), R7.2, RN1.1 (common), U2.5 (V_{SS}); no longer JP1.1 (A), R2.2, R3.2, R4.2, SW1.1 (A)
- net RX: now also J2.3 (Pin_3)
- net SCL: now also R13.1
- net SDA: now also R14.1
- net TX: now also J2.2 (Pin_2)
- net BMS/B+ renamed V_{BAT}
- net V_{BAT}: now also C6.1, U2.10 (V_{BAT}), U2.9 (V_{BAT})
- net BMS/B-: no longer names the net of BT1.2 (-)
- net BMS/B-: now also JP1.1 (A), SW1.1 (A)
- net IO10 renamed IRQ_{ON}
- net IRQ_{ON}: now also SW3.1, U4.11 (D0), RN1.9 (R8)
- net IO18 renamed D-
- net D-: now also J1.A7 (D-), J1.B7 (D-)
- net IO19 renamed D+
- net D+: now also J1.A6 (D+), J1.B6 (D+)
- net IO2: no longer names the net of R10.2, U3.5 (IO2)
- net IO8: no longer names the net of R11.2, U3.22 (IO8)
- net IO9: no longer names the net of JP2.1 (A), U3.23 (IO9)
- removed net PD0: R2.1, SW3.1, U4.11 (D0)
- net PD1: no longer names the net of SW4.1, U4.12 (D1)
- net PD1: now also RN1.8 (R7); no longer R3.1
- net PD2: no longer names the net of SW6.1, U4.13 (D2)
- net PD2: now also RN1.7 (R6); no longer R4.1
- net PD3: no longer names the net of SW9.1, U4.14 (D3)
- net PD3: now also RN1.6 (R5); no longer R5.1
- net PD4: no longer names the net of SW5.1, U4.3 (D4)
- net PD4: now also RN1.3 (R2); no longer R6.1
- net PD5: no longer names the net of SW7.1, U4.4 (D5)
- net PD5: now also RN1.4 (R3); no longer R8.1
- net PD6: no longer names the net of SW10.1, U4.5 (D6)
- net PD6: now also RN1.5 (R4)
- net PD7: no longer names the net of SW8.1, U4.6 (D7)
- net PD7: now also RN1.2 (R1)
- new net: D1.3 (BK), R2.1
- new net: R2.2, U2.4 (STAT2)
- new net: J1.A5 (CC1), R7.1
- new net: J1.B5 (CC2), R8.1
- new net: R5.1, U2.6 (PROG)
- new net: D1.1 (RK), R4.2
- new net: D1.2 (GK), R3.1
- new net: R4.1, U2.3 (STAT1)
- new net: R3.2, U2.7 (~{PG})
- new net: R6.1, U2.8 (THERM)
- new net: R12.1, U5.12 (SDO/ADDR)
- new net V_{BUS}: C5.1, D1.4 (BA), D1.5 (GA), D1.6 (RA), J1.A4 (VBUS), J1.A9 (VBUS), J1.B4 (VBUS), J1.B9 (VBUS), U2.1 (V_{DD}), U2.2 (V_{DD})
- now unconnected: U3.10 (NC_4), U3.15 (NC_5), U3.17 (NC_6), U3.24 (NC_7), U3.25 (NC_8), U3.28 (NC_9), U3.29 (NC_10), U3.32 (NC_11), U3.33 (NC_12), U3.34 (NC_13), U3.35 (NC_14), U3.4 (NC_1), U3.7 (NC_2), U3.9 (NC_3)
Other:
- removed sheet BMS
- note added: "I2C pull-up"
- note added: "accelerometer"
- note added: "battery charger"
- note added: "microcontroller"
- note removed: "Accelerometer"
- note removed: "either or"
- moved on the sheet: C1, C11, C2, JP1, JP2, L1, R1, R10, R11, R15, SW1, SW10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

Commit message: 2024-04-18
Parts:
- added R16, R18: LDR, OptoDevice:R_LDR_5.0x4.1mm_P3mm_Vertical, symbol Device:R_Photo
- added R17, R19: 10K, Resistor_SMD:R_0603_1608Metric_Pad0.98x0.95mm_HandSolder, symbol Device:R
- added RN2: YC248-JR-074K7L, footprints:RES_YC248_4X1P6_YAG, symbol Custom:R_Array08
- added TP1: TestPoint, TestPoint:TestPoint_Pad_D1.5mm, symbol Connector:TestPoint
- C1, C10, C11, C12, C2, C3, C4, C5, C6: footprint (none) -> Capacitor_SMD:C_0603_1608Metric_Pad1.08x0.95mm_HandSolder
- C7, C8, C9: footprint Custom:C_0603_HandSolder_ValuePrinted -> Capacitor_SMD:C_0603_1608Metric_Pad1.08x0.95mm_HandSolder
- D1: symbol Device:LED_RGB -> Device:LED_ARGB
- JP2: footprint Connector_PinHeader_2.00mm:PinHeader_1x02_P2.00mm_Vertical -> Jumper:SolderJumper-2_P1.3mm_Open_TrianglePad1.0x1.5mm
- L1: value 2.2uH -> LPS4012-222MRC; footprint (none) -> Custom:L_Coilcraft_LPS4012
- R1, R12, R13, R14, R2, R3, R4, R5, R6, R7, R8: footprint (none) -> Resistor_SMD:R_0603_1608Metric_Pad0.98x0.95mm_HandSolder
- R10, R11, R9: footprint Custom:R_0603_HandSolder_ValuePrinted -> Resistor_SMD:R_0603_1608Metric_Pad0.98x0.95mm_HandSolder
- R15: value ~24K -> 24K; footprint (none) -> Resistor_SMD:R_0603_1608Metric_Pad0.98x0.95mm_HandSolder
- RN1: symbol Device:R_Network08 -> Custom:R_Array08
Connections:
- net +3V3: now also R16.1, R18.1, RN2.3 (R2), RN2.6 (R5); no longer DS1.11 (BS1), DS1.13 (~{CS})
- net CP: now also R11.2, U3.22 (IO8); no longer U3.18 (IO4)
- net GND: now also RN1.2 (R1), RN1.3 (R2), RN1.4 (R3), RN1.5 (R4), RN1.6 (R5), RN1.7 (R6), RN1.8 (R7), R17.2, R19.2, RN2.4 (R3), RN2.7 (R6), RN2.8 (R7); no longer DS1.12 (BS2), DS1.14 (~{RES}), DS1.15 (D/~{C})
- net INT1: now also U3.6 (IO3); no longer U3.20 (IO6)
- net INT2: now also U3.18 (IO4); no longer U3.21 (IO7)
- net Q7: now also R10.2, U3.5 (IO2); no longer U3.6 (IO3)
- net SCL: now also U3.19 (IO5); no longer U3.12 (IO0)
- net SDA: now also U3.20 (IO6); no longer U3.13 (IO1)
- net SH/~{LD}: now also U3.21 (IO7); no longer U3.19 (IO5)
- net V_{BUS}: now also D1.1 (A); no longer D1.4 (BA), D1.5 (GA), D1.6 (RA)
- net at SW9.1, U4.14 (D3): now also RN1.12 (R8); no longer RN1.6 (R5)
- net at SW5.1, U4.3 (D4): now also RN1.15 (R8); no longer RN1.3 (R2)
- net at R2.1: now also D1.4 (BK); no longer D1.3 (BK)
- net ~{PG}: now reaches R2.2, U2.4 (STAT2)
- net at SW6.1, U4.13 (D2): now also RN1.11 (R8); no longer RN1.7 (R6)
- net at SW8.1, U4.6 (D7): now also RN1.16 (R8); no longer RN1.2 (R1)
- net at R5.1, U2.6 (PROG): now also TP1.1
- net at R4.2: now also D1.2 (RK); no longer D1.1 (RK)
- net at R3.1: now also D1.3 (GK); no longer D1.2 (GK)
- net V_{BAT}-: now reaches BT1.2 (-), JP1.1 (A), SW1.1 (A)
- net at SW4.1, U4.12 (D1): now also RN1.10 (R8); no longer RN1.8 (R7)
- net at SW7.1, U4.4 (D5): now also RN1.14 (R8); no longer RN1.4 (R3)
- net at SW10.1, U4.5 (D6): now also RN1.13 (R8); no longer RN1.5 (R4)
- net STAT1: now reaches R4.1, U2.3 (STAT1)
- net STAT2: now reaches R3.2, U2.7 (~{PG})
- net V_{BAT} renamed V_{BAT}+
- new net: DS1.11 (BS1), RN2.14 (R8)
- new net: DS1.12 (BS2), RN2.13 (R8)
- new net: DS1.13 (~{CS}), RN2.11 (R8)
- new net: DS1.14 (~{RES}), RN2.10 (R8)
- new net: DS1.15 (D/~{C}), RN2.9 (R8)
- new net LDR1: R16.2, R17.1, U3.12 (IO0)
- new net LDR2: R18.2, R19.1, U3.13 (IO1)
- no-connect marks 19 -> 25
Other:
- note added: "LDRs"
- note added: "USB"
- note added: "^"
- note added: "peak: 140uA"
- note added: "peak: 500mA"
- note added: "peak: 50mA"
- note added: "peak: 80uA"
- note added: "v"
- moved on the sheet: C2, L1, R5
