File: LED driver/LED driver.kicad_sch (KiCad schematic)
At the start: 45 parts, among them J1 Conn_Aux, J2 Conn_UART, J3 Conn_LED, J4 Conn_VCC_Alt, J5 Conn_VCC, Q1 ZXMN3A01F, Q2 ZXMN3A01F, Q3 ZXMN3A01F, Q4 ZXMN3A01F, Q5 ZXMN3A01F, SW1 SW_Push, U1 ESP32-C3-WROOM-02, U2 MP2359

Commit message: 2024-04-13
Parts:
- J2: renamed from J5; footprint Connector_BarrelJack:BarrelJack_GCT_DCJ200-10-A_Horizontal -> Custom:BarrelJack_GCT_DCJ200-10-A_Horizontal
- R12, R13: value 10K -> 100K
- U1: value ESP32-C3-WROOM-02 -> ESP32-C3-MINI-1-N4; footprint RF_Module:ESP32-C3-WROOM-02 -> ESP32C3MINI1N4; symbol Custom:ESP32-C3-WROOM-02 -> Custom:ESP32-C3-MINI-1-N4; Height (none) -> 2.55; Manufacturer_Name (none) -> Espressif Systems; Manufacturer_Part_Number (none) -> ESP32-C3-MINI-1-N4; Mouser Part Number (none) -> 356-ESP32-C3-MINI1N4; Mouser Price/Stock (none) -> https://www.mouser.co.uk/ProductDetail/Espressif-Systems/ES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
- renumbered J4 to J1, J2 to J5, J1 to J6
Connections:
- net +3.3V: now also U1.3 (3V3); no longer U1.1 (VDD)
- net GND: now also U1.1 (GND), U1.11 (GND_3), U1.14 (GND_4), U1.2 (GND_2), U1.36 (GND_5), U1.37 (GND_6), U1.38 (GND_7), U1.39 (GND_8), U1.40 (GND_9), U1.41 (GND_10), U1.42 (GND_11), U1.43 (GND_12), U1.44 (GND_13), U1.45 (GND_14), U1.46 (GND_15), U1.47 (GND_16), U1.48 (GND_17), U1.49 (GND_18), U1.50 (GND_19), U1.51 (GND_20), U1.52 (GND_21), U1.53 (GND_22), U1.54 (GND_23), U1.55 (GND_24), U1.56 (GND_25), U1.57 (GND_26), U1.58 (GND_27), U1.59 (GND_28), U1.60 (GND_29), U1.61 (GND_30); no longer U1.19 (GND), U1.9 (GND)
- net IO9: now also U1.23 (IO9); no longer J6.8 (Pin_8), U1.8 (IO9)
- net PWM_B: now also U1.20 (IO6); no longer R12.2, U1.16 (IO2)
- net PWM_G: now also U1.19 (IO5); no longer U1.17 (IO1)
- net PWM_W: now also U1.21 (IO7); no longer U1.15 (IO3)
- net PWM_WW: now also R13.2, U1.22 (IO8); no longer U1.14 (IO19)
- net RX: now also R14.1, U1.30 (RXD0); no longer J5.3 (Pin_3), R14.2
- net TX: now also R15.1, U1.31 (TXD0); no longer J5.2 (Pin_2), R15.2
- net at U1.10 (NC_4): now also U1.15 (NC_5), U1.17 (NC_6), U1.24 (NC_7), U1.25 (NC_8), U1.28 (NC_9), U1.29 (NC_10), U1.32 (NC_11), U1.33 (NC_12), U1.34 (NC_13), U1.35 (NC_14), U1.4 (NC_1), U1.7 (NC_2), U1.9 (NC_3)
- net IO0: now reaches U1.12 (IO0)
- net IO0: now also J6.3 (Pin_3); no longer R15.1
- net IO1: now reaches U1.13 (IO1)
- net IO1: now also J6.4 (Pin_4)
- net at C2.2, R11.2, SW1.2: now also U1.8 (EN); no longer U1.2 (EN)
- removed net IO4: J6.3 (Pin_3), U1.3 (IO4)
- removed net IO5: J6.4 (Pin_4), U1.4 (IO5)
- net IO6 renamed IO2
- net IO2: now also R12.2
- net IO7 renamed IO3
- removed net IO8: J6.7 (Pin_7), R13.2, U1.7 (IO8)
- new net: J5.2 (Pin_2), R15.2
- new net: J5.3 (Pin_3), R14.2
- new net IO18: J6.7 (Pin_7), U1.26 (IO18)
- new net IO19: J6.8 (Pin_8), U1.27 (IO19)
- no-connect marks 3 -> 2
Other:
- moved on the sheet: JP1, JP2, R12, R13, R14, R15

Commit message: 2024-06-04 001
Parts:
- removed J1: Conn_VCC_Alt, TerminalBlock_Phoenix:TerminalBlock_Phoenix_MKDS-1,5-2_1x02_P5.00mm_Horizontal, symbol Connector:Screw_Terminal_01x02
- removed R14, R15: 0, Resistor_SMD:R_0603_1608Metric_Pad0.98x0.95mm_HandSolder, symbol Device:R_Small
- added JP2: Boot Mode 2, Connector_PinHeader_2.00mm:PinHeader_1x03_P2.00mm_Vertical, symbol Jumper:Jumper_3_Bridged12
- added TP1: PWM_W, TestPoint:TestPoint_Loop_D2.50mm_Drill1.0mm, symbol Connector:TestPoint
- added TP2: PWM_B, TestPoint:TestPoint_Loop_D2.50mm_Drill1.0mm, symbol Connector:TestPoint
- added TP3: PWM_R, TestPoint:TestPoint_Loop_D2.50mm_Drill1.0mm, symbol Connector:TestPoint
- added TP4: PWM_G, TestPoint:TestPoint_Loop_D2.50mm_Drill1.0mm, symbol Connector:TestPoint
- added TP5: PWM_WW, TestPoint:TestPoint_Loop_D2.50mm_Drill1.0mm, symbol Connector:TestPoint
- C1, C2, C3, C6: footprint Custom:C_0603_HandSolder_ValuePrinted -> Capacitor_SMD:C_0603_1608Metric
- C4: renamed from C5; footprint Custom:C_0603_HandSolder_ValuePrinted -> Capacitor_SMD:C_0603_1608Metric
- C5: renamed from C4; footprint Custom:C_0603_HandSolder_ValuePrinted -> Capacitor_SMD:C_0603_1608Metric
- D2: value B230A -> B230-13-F; footprint Diode_SMD:D_SMA -> Diode_SMD:D_SMB
- D3: renamed from D1; footprint Diode_SMD:D_0603_1608Metric_Pad1.05x0.95mm_HandSolder -> Diode_SMD:D_0603_1608Metric
- J1: renamed from J2; symbol Connector:Barrel_Jack_Switch -> Connector:Screw_Terminal_01x02
- J4: renamed from J5; footprint Connector_PinHeader_2.54mm:PinHeader_1x04_P2.54mm_Vertical -> Connector_PinHeader_2.00mm:PinHeader_1x04_P2.00mm_Vertical; symbol Connector_Generic:Conn_01x04 -> Connector:Conn_01x04_Pin
- JP1: value Boot_Mode -> Boot Mode 1
- L1: footprint Inductor_SMD:L_1210_3225Metric_Pad1.42x2.65mm_HandSolder -> Inductor_SMD:L_1210_3225Metric
- Q1, Q2, Q3, Q4, Q5: footprint Package_TO_SOT_SMD:SOT-23 -> Custom:SOT-23
- R1, R10, R11, R12, R2, R3, R4, R5, R6, R7, R8, R9: footprint Custom:R_0603_HandSolder_ValuePrinted -> Resistor_SMD:R_0603_1608Metric
- R13: value 100K -> 4.7K; footprint Custom:R_0603_HandSolder_ValuePrinted -> Resistor_SMD:R_0603_1608Metric
- R14: renamed from R16; footprint Custom:R_0603_HandSolder_ValuePrinted -> Resistor_SMD:R_0603_1608Metric
- R15: renamed from R17; footprint Custom:R_0603_HandSolder_ValuePrinted -> Resistor_SMD:R_0603_1608Metric
- R16: renamed from R19; footprint Custom:R_0603_HandSolder_ValuePrinted -> Resistor_SMD:R_0603_1608Metric
- R17: renamed from R18; footprint Custom:R_0603_HandSolder_ValuePrinted -> Resistor_SMD:R_0603_1608Metric
- U1: footprint ESP32C3MINI1N4 -> ESP32-C3-MINI-1-N4:ESP32C3MINI1N4
- renumbered D3 to D1, J3 to J2, J6 to J3, JP2 to JP3
Connections:
- net GND: now also J1.1 (Pin_1), J4.4 (Pin_4); no longer J1.2, J4.1 (Pin_1)
- net PWM_B: now also TP2.1
- net PWM_G: now also TP4.1
- net PWM_R: now also TP3.1
- net PWM_W: now also TP1.1
- net PWM_WW: now also JP2.1 (A), TP5.1; no longer R13.2, U1.22 (IO8)
- net RX: now also J4.2 (Pin_2)
- net TX: now also J4.3 (Pin_3)
- net at F1.2: now also J1.2 (Pin_2); no longer J1.1
- net at JP3.2 (B): now also J4.1 (Pin_1); no longer J4.4 (Pin_4)
- new net: JP2.2 (C), U1.22 (IO8)
- new net: JP2.3 (B), R13.2
- no-connect marks 2 -> 1
Other:
- moved on the sheet: C2, C6, D1, F1, J3, JP1, JP3, L1, R12, R15, R16, SW1

Commit message: 2024-06-04 002
Parts:
- added J5: PWR_AUX, Connector_PinHeader_2.54mm:PinHeader_1x03_P2.54mm_Vertical, symbol Connector:Conn_01x03_Socket
- J1: footprint Custom:BarrelJack_GCT_DCJ200-10-A_Horizontal -> TerminalBlock_Phoenix:TerminalBlock_Phoenix_MKDS-1,5-2_1x02_P5.00mm_Horizontal
Connections:
- net +3.3V: now also J5.3 (Pin_3)
- net GND: now also J5.2 (Pin_2)
- net VCC: now also J5.1 (Pin_1)

Commit message: 2024-06-05
Parts:
- D3: footprint Diode_SMD:D_0603_1608Metric -> Diode_SMD:D_0603_1608Metric_Pad1.05x0.95mm_HandSolder; now not fitted
- F1: value 24VDC 10A -> 24VDC 5A
- R17: footprint Resistor_SMD:R_0603_1608Metric -> Resistor_SMD:R_0603_1608Metric_Pad0.98x0.95mm_HandSolder; now not fitted
Changed lines of the file:
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@@
 			)
 		)
-		(property "Value" "24VDC 10A"
+		(property "Value" "24VDC 5A"
 			(at 46.99 152.4 90)
 			(effects
@@
 		(in_bom yes)
 		(on_board yes)
-		(dnp no)
+		(dnp yes)
 		(fields_autoplaced yes)
 		(property "Reference" "D3"
@@
 			)
 		)
-		(property "Footprint" "Diode_SMD:D_0603_1608Metric"
+		(property "Footprint" "Diode_SMD:D_0603_1608Metric_Pad1.05x0.95mm_HandSolder"
 			(at 166.37 152.4 0)
 			(effects
@@
 		(in_bom yes)
 		(on_board yes)
-		(dnp no)
+		(dnp yes)
 		(property "Reference" "R17"
 			(at 168.148 163.8299 0)
@@
 			)
 		)
-		(property "Footprint" "Resistor_SMD:R_0603_1608Metric"
+		(property "Footprint" "Resistor_SMD:R_0603_1608Metric_Pad0.98x0.95mm_HandSolder"
 			(at 168.148 165.1 90)
 			(effects

Commit message: 2024-11-23
Parts:
- removed JP3: SolderJumper_2_Open, Jumper:SolderJumper-2_P1.3mm_Open_RoundedPad1.0x1.5mm, symbol Jumper:SolderJumper_2_Open
- J4: footprint Connector_PinHeader_2.00mm:PinHeader_1x04_P2.00mm_Vertical -> Connector_PinHeader_2.54mm:PinHeader_1x04_P2.54mm_Vertical
- JP1: footprint Connector_PinHeader_2.00mm:PinHeader_1x02_P2.00mm_Vertical -> Connector_PinHeader_2.54mm:PinHeader_1x02_P2.54mm_Vertical
- JP2: footprint Connector_PinHeader_2.00mm:PinHeader_1x03_P2.00mm_Vertical -> Connector_PinHeader_2.54mm:PinHeader_1x03_P2.54mm_Vertical
Connections:
- net +3.3V: now also J4.1 (Pin_1)
- net GND: now also J4.2 (Pin_2); no longer J4.4 (Pin_4)
- net RX: now also J4.3 (Pin_3); no longer J4.2 (Pin_2)
- net TX: now also J4.4 (Pin_4); no longer J4.3 (Pin_3)
Changed lines of the file:
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@@
 	(wire
 		(pts
-			(xy 34.29 111.76) (xy 31.75 111.76)
+			(xy 34.29 106.68) (xy 31.75 106.68)
 		)
 		(stroke
@@
 	(wire
 		(pts
-			(xy 31.75 109.22) (xy 39.37 109.22)
+			(xy 31.75 111.76) (xy 39.37 111.76)
 		)
 		(stroke
@@
 	(wire
 		(pts
-			(xy 34.29 91.44) (xy 34.29 93.98)
+			(xy 34.29 101.6) (xy 34.29 104.14)
 		)
 		(stroke
@@
 	(wire
 		(pts
-			(xy 34.29 101.6) (xy 34.29 104.14)
-		)
-		(stroke
-			(width 0)
-			(type default)
-		)
-	)
-	(wire
-		(pts
 			(xy 105.41 69.85) (xy 105.41 68.58)
 		)
@@
 	(wire
 		(pts
-			(xy 34.29 111.76) (xy 34.29 114.3)
+			(xy 34.29 106.68) (xy 34.29 114.3)
 		)
 		(stroke
@@
 	(wire
 		(pts
-			(xy 31.75 106.68) (xy 39.37 106.68)
+			(xy 31.75 109.22) (xy 39.37 109.22)
 		)
 		(stroke
@@
 	)
 	(label "RX"
-		(at 39.37 106.68 180)
+		(at 39.37 109.22 180)
 		(fields_autoplaced yes)
 		(effects
@@
 	)
 	(label "TX"
-		(at 39.37 109.22 180)
+		(at 39.37 111.76 180)
 		(fields_autoplaced yes)
 		(effects
@@
 			)
 		)
-		(property "Footprint" "Connector_PinHeader_2.00mm:PinHeader_1x04_P2.00mm_Vertical"
+		(property "Footprint" "Connector_PinHeader_2.54mm:PinHeader_1x04_P2.54mm_Vertical"
 			(at 26.67 106.68 0)
 			(effects
@@
 	(symbol
 		(lib_id "power:+3.3V")
-		(at 34.29 91.44 0)
+		(at 34.29 101.6 0)
 		(unit 1)
 		(exclude_from_sim no)
@@
 		(fields_autoplaced yes)
 		(property "Reference" "#PWR025"
-			(at 34.29 95.25 0)
+			(at 34.29 105.41 0)
 			(effects
 				(font
@@
 		)
 		(property "Value" "+3.3V"
-			(at 36.83 90.1699 0)
+			(at 36.83 100.3299 0)
 			(effects
 				(font
@@
 		)
 		(property "Footprint" ""
-			(at 34.29 91.44 0)
+			(at 34.29 101.6 0)
 			(effects
 				(font
@@
 		)
 		(property "Datasheet" ""
-			(at 34.29 91.44 0)
+			(at 34.29 101.6 0)
 			(effects
 				(font
@@
 		)
 		(property "Description" "Power symbol creates a global label with name \"+3.3V\""
-			(at 34.29 91.44 0)
+			(at 34.29 101.6 0)
 			(effects
 				(font
@@
 	)
 	(symbol
-		(lib_id "Jumper:SolderJumper_2_Open")
-		(at 34.29 97.79 270)
-		(unit 1)
-		(exclude_from_sim yes)
-		(in_bom no)
-		(on_board yes)
-		(dnp no)
-		(property "Reference" "JP3"
-			(at 36.83 97.7899 90)
-			(effects
-				(font
-					(size 1.27 1.27)
-				)
-				(justify left)
-			)
-		)
-		(property "Value" "SolderJumper_2_Open"
-			(at 36.83 99.0599 90)
-			(effects
-				(font
-					(size 1.27 1.27)
-				)
-				(justify left)
-				(hide yes)
-			)
-		)
-		(property "Footprint" "Jumper:SolderJumper-2_P1.3mm_Open_RoundedPad1.0x1.5mm"
-			(at 34.29 97.79 0)
-			(effects
-				(font
-					(size 1.27 1.27)
-				)
-				(hide yes)
-			)
-		)
-		(property "Datasheet" "~"
-			(at 34.29 97.79 0)
-			(effects
-				(font
-					(size 1.27 1.27)
-				)
-				(hide yes)
-			)
-		)
-		(property "Description" "Solder Jumper, 2-pole, open"
-			(at 34.29 97.79 0)
-			(effects
-				(font
-					(size 1.27 1.27)
-				)
-				(hide yes)
-			)
-		)
-		(pin "1"
-		)
-		(pin "2"
-		)
-		(instances
-			(project "LED driver"
-				(path "/3b6d8f14-65dd-401e-abe3-3efb7da28af6"
-					(reference "JP3")
-					(unit 1)
-				)
-			)
-		)
-	)
-	(symbol
 		(lib_id "power:+3.3V")
 		(at 166.37 146.05 0)
@@
 			)
 		)
-		(property "Footprint" "Connector_PinHeader_2.00mm:PinHeader_1x02_P2.00mm_Vertical"
+		(property "Footprint" "Connector_PinHeader_2.54mm:PinHeader_1x02_P2.54mm_Vertical"
 			(at 45.72 72.39 0)
 			(effects
@@
 			)
 		)
-		(property "Footprint" "Connector_PinHeader_2.00mm:PinHeader_1x03_P2.00mm_Vertical"
+		(property "Footprint" "Connector_PinHeader_2.54mm:PinHeader_1x03_P2.54mm_Vertical"
 			(at 100.33 85.09 0)
 			(effects

Commit message: 2024-11-24 (sub-par pcb)
Parts:
- removed J4: Conn_UART, Connector_PinHeader_2.54mm:PinHeader_1x04_P2.54mm_Vertical, symbol Connector:Conn_01x04_Pin
- removed JP1: Boot Mode 1, Connector_PinHeader_2.54mm:PinHeader_1x02_P2.54mm_Vertical, symbol Jumper:Jumper_2_Open
- removed JP2: Boot Mode 2, Connector_PinHeader_2.54mm:PinHeader_1x03_P2.54mm_Vertical, symbol Jumper:Jumper_3_Bridged12
- removed R13: 4.7K, Resistor_SMD:R_0603_1608Metric, symbol Device:R
- removed TP1: PWM_W, TestPoint:TestPoint_Loop_D2.50mm_Drill1.0mm, symbol Connector:TestPoint
- removed TP2: PWM_B, TestPoint:TestPoint_Loop_D2.50mm_Drill1.0mm, symbol Connector:TestPoint
- removed TP3: PWM_R, TestPoint:TestPoint_Loop_D2.50mm_Drill1.0mm, symbol Connector:TestPoint
- removed TP4: PWM_G, TestPoint:TestPoint_Loop_D2.50mm_Drill1.0mm, symbol Connector:TestPoint
- removed TP5: PWM_WW, TestPoint:TestPoint_Loop_D2.50mm_Drill1.0mm, symbol Connector:TestPoint
- added J4: USB_B_Mini, Connector_USB:USB_Mini-B_AdamTech_MUSB-B5-S-VT-TSMT-1_SMD_Vertical, symbol Connector:USB_B_Mini
- added J6: Conn_VCC, Connector_JST:JST_VH_B2PS-VH_1x02_P3.96mm_Horizontal, symbol Connector:Conn_01x02_Pin
- added JP1: VBUS_to_VCC, Connector_PinHeader_2.54mm:PinHeader_1x02_P2.54mm_Vertical, symbol Jumper:Jumper_2_Small_Open
- J1: value Conn_VCC -> Conn_VCC_screw; now not fitted
- J2: footprint footprints:CON_532540670_MOL -> Connector_JST:JST_VH_B6PS-VH_1x06_P3.96mm_Horizontal
- U1: footprint ESP32-C3-MINI-1-N4:ESP32C3MINI1N4 -> ESP32C3MINI1N4
Connections:
- net B: now also J2.5 (Pin_5); no longer J2.3 (Pin_3)
- net G: now also J2.3 (Pin_3); no longer J2.5 (Pin_5)
- net GND: now also J4.5 (GND), J4.6 (Shield), J6.1 (Pin_1)
- net IO0: now also J3.8 (Pin_8); no longer J3.3 (Pin_3)
- net IO1: now also J3.7 (Pin_7); no longer J3.4 (Pin_4)
- net IO2: now also J3.4 (Pin_4); no longer J3.5 (Pin_5)
- net IO3: now also J3.3 (Pin_3); no longer J3.6 (Pin_6)
- net PWM_B: now also U1.21 (IO7); no longer U1.20 (IO6)
- net PWM_R: now also U1.20 (IO6); no longer U1.18 (IO4)
- net PWM_W: now also U1.22 (IO8); no longer U1.21 (IO7)
- net PWM_WW: now also U1.18 (A1_4/IO4)
- net VCC: now also JP1.2 (B)
- net W: now also J2.6 (Pin_6); no longer J2.2 (Pin_2)
- net WW: now also J2.2 (Pin_2); no longer J2.6 (Pin_6)
- net at F1.2, J1.2 (Pin_2): now also J6.2 (Pin_2)
- net IO18 renamed USB_D-
- net USB_D-: now also J4.2 (D-); no longer J3.7 (Pin_7)
- net IO19 renamed USB_D+
- net USB_D+: now also J4.3 (D+); no longer J3.8 (Pin_8)
- net IO9: no longer names the net of U1.23 (IO9)
- net RX renamed IO20
- net IO20: now also J3.5 (Pin_5)
- net TX renamed IO21
- net IO21: now also J3.6 (Pin_6)
- new net: J4.1 (VBUS), JP1.1 (A)
- no-connect marks 1 -> 3
Other:
- moved on the sheet: C2, J2, R11, R12, SW1
