File: LED driver/LED driver.kicad_pcb (KiCad board)
At the start: 2 copper layers, 57.5 x 41 mm, 45 parts, among them J1 Conn_VCC_Alt, J2 Conn_VCC, J3 Conn_LED, J4 Conn_Boot_Mode, J5 Conn_UART, J6 Conn_Aux, Q1 ZXMN3A01F, Q2 ZXMN3A01F, Q3 ZXMN3A01F, Q4 ZXMN3A01F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

Commit message: 2024-04-13
Parts:
- removed J4: Conn_Boot_Mode, Connector_PinHeader_2.54mm:PinHeader_1x02_P2.54mm_Vertical
- removed R20: 300, Custom:R_0603_HandSolder_ValuePrinted
- added JP1: Boot_Mode, Connector_PinHeader_2.00mm:PinHeader_1x02_P2.00mm_Vertical, F.Cu at (151.7, 73.4)
- added JP2: SolderJumper_2_Open, Jumper:SolderJumper-2_P1.3mm_Open_RoundedPad1.0x1.5mm, F.Cu at (152.0, 67.5)
- C1: value 0.1uF -> 10uF
- C2, C3: value 10uF -> 0.1uF
- C4: value 0.1uF -> 10nF
- C5: value 10nF -> 10uF
- D1: value SMF24A -> PWR_LED; footprint Diode_SMD:D_SMF -> Diode_SMD:D_0603_1608Metric_Pad1.05x0.95mm_HandSolder
- D3: value PWR_LED -> SMF24A; footprint Diode_SMD:D_0603_1608Metric_Pad1.05x0.95mm_HandSolder -> Diode_SMD:D_SMF
- J2: footprint Connector_BarrelJack:BarrelJack_GCT_DCJ200-10-A_Horizontal -> Custom:BarrelJack_GCT_DCJ200-10-A_Horizontal
- R11: value 0 -> 10K; footprint Resistor_SMD:R_0603_1608Metric_Pad0.98x0.95mm_HandSolder -> Custom:R_0603_HandSolder_ValuePrinted
- R12: value 10K -> 100K
- R13: value 0 -> 100K; footprint Resistor_SMD:R_0603_1608Metric_Pad0.98x0.95mm_HandSolder -> Custom:R_0603_HandSolder_ValuePrinted
- R15: value 10K -> 0; footprint Custom:R_0603_HandSolder_ValuePrinted -> Resistor_SMD:R_0603_1608Metric_Pad0.98x0.95mm_HandSolder
- R17: value 10K -> 49.9K
- R18: value 49.9K -> 300
- U1: value ESP32-C3-WROOM-02 -> ESP32-C3-MINI-1-N4; footprint RF_Module:ESP32-C3-WROOM-02 -> ESP32-C3-MINI-1-N4:ESP32C3MINI1N4
- moved R17 31.1 mm to (121.9, 59.8), turned to 0 degrees
- moved R15 23.8 mm to (152.0, 62.2), turned to 0 degrees
- moved R11 23.5 mm to (131.9, 73.0), turned to 0 degrees
- moved D1 23.2 mm to (129.1, 58.4), turned to 180 degrees
- moved R14 16.0 mm to (152.0, 64.0), turned to 180 degrees
- moved R12 13.7 mm to (132.8, 65.9)
- moved C2 12.1 mm to (132.0, 71.2), turned to 0 degrees
- moved SW1 11.4 mm to (132.0, 68.5)
- moved F1 11.3 mm to (114.3, 61.3), turned to 180 degrees
- moved D3 8.84 mm to (114.3, 66.6)
- moved R18 7.92 mm to (125.6, 58.4)
- moved C1 7.90 mm to (133.7, 63.3), turned to -90 degrees
- moved J3 7.16 mm to (146.8, 88.5)
- moved Q1 7.16 mm to (139.9, 85.5)
- moved Q2 7.16 mm to (133.4, 85.5)
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Connections:
- net /IO7 renamed /IO3
- C1 pad 2: Net-(U1-EN) -> +3.3V
- C2 pad 1: VCC -> GND
- C2 pad 2: GND -> Net-(U1-EN)
- C4 pad 1: GND -> Net-(U2-BST)
- C4 pad 2: +3.3V -> Net-(D2-K)
- C5 pad 1: Net-(U2-BST) -> VCC
- C5 pad 2: Net-(D2-K) -> GND
- D1 pad 1: VCC -> +3.3V
- D1 pad 2: GND -> Net-(D1-A)
- D3 pad 1: +3.3V -> VCC
- D3 pad 2: Net-(D3-A) -> GND
- J5 pad 2: /TX -> Net-(J5-Pin_2)
- J5 pad 3: /RX -> Net-(J5-Pin_3)
- J6 pad 3: /IO4 -> /IO0
- J6 pad 4: /IO5 -> /IO1
- J6 pad 5: /IO6 -> /IO2
- J6 pad 7: /IO8 -> /IO18
- J6 pad 8: /IO9 -> /IO19
- R11 pad 1: Net-(J5-Pin_4) -> +3.3V
- R11 pad 2: +3.3V -> Net-(U1-EN)
- R12 pad 2: /IO8 -> /IO2
- R13 pad 1: Net-(U1-RXD) -> +3.3V
- R13 pad 2: /RX -> /PWM_WW
- R14 pad 1: Net-(U1-TXD) -> /RX
- R14 pad 2: /TX -> Net-(J5-Pin_3)
- R15 pad 1: +3.3V -> /TX
- R15 pad 2: Net-(U1-EN) -> Net-(J5-Pin_2)
- R17 pad 1: +3.3V -> Net-(U2-FB)
- R17 pad 2: /PWM_B -> +3.3V
- R18 pad 1: Net-(U2-FB) -> GND
- R18 pad 2: +3.3V -> Net-(D1-A)
- U1 pad 1: +3.3V -> GND
- U1 pad 11: Net-(U1-RXD) -> GND
- U1 pad 12: Net-(U1-TXD) -> /IO0
- U1 pad 13: unconnected-(U1-IO18-Pad13) -> /IO1
- U1 pad 14: /PWM_WW -> GND
- U1 pad 15: /PWM_W -> unconnected-(U1-NC_5-Pad15)
- U1 pad 16: /PWM_B -> unconnected-(U1-IO10-Pad16)
- U1 pad 17: /PWM_G -> unconnected-(U1-NC_6-Pad17)
- U1 pad 19: GND -> /PWM_G
- U1 pad 2: Net-(U1-EN) -> GND
- U1 pad 3: /IO4 -> +3.3V
- U1 pad 4: /IO5 -> unconnected-(U1-NC_1-Pad4)
- U1 pad 5: /IO6 -> /IO2
- U1 pad 7: /IO8 -> unconnected-(U1-NC_2-Pad7)
- U1 pad 8: /IO9 -> Net-(U1-EN)
- U1 pad 9: GND -> unconnected-(U1-NC_3-Pad9)
Routing:
- net GND: track 112.1 -> 52.4 mm, vias 5 -> 0
- net /IO0: track 0.00 -> 51.8 mm, vias 0 -> 1
- net /IO19: track 0.00 -> 50.6 mm, vias 0 -> 1
- net /IO18: track 0.00 -> 49.3 mm, vias 0 -> 1
- net /IO1: track 0.00 -> 48.6 mm, vias 0 -> 1
- net /IO9: track 53.7 -> 6.64 mm, vias 1 -> 0
- net /IO8: track 46.8 -> 0.00 mm, vias 1 -> 0
- net /IO2: track 0.00 -> 45.7 mm, vias 0 -> 1
- net /IO4: track 41.3 -> 0.00 mm, vias 1 -> 0
- net /IO5: track 41.2 -> 0.00 mm, vias 1 -> 0
- net /IO6: track 39.1 -> 0.00 mm, vias 1 -> 0
- net +3.3V: track 143.0 -> 114.4 mm, vias 3 -> 2
- net /PWM_R: track 39.7 -> 19.9 mm, vias 2 -> 0
- net /PWM_B: track 31.1 -> 14.4 mm, vias 2 -> 0
- net /PWM_G: track 44.7 -> 29.8 mm
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Other:
- board size 57.5 x 41 mm -> 60 x 40 mm
- board text removed: "BOOT MODE"
- board text removed: "JLCJLCJLCJLC"
- board text removed: "ON"
- board text removed: "RST"

Commit message: 2024-06-04 001
Parts:
- removed J5: Conn_UART, Connector_PinHeader_2.54mm:PinHeader_1x04_P2.54mm_Vertical
- removed J6: Conn_Aux, Connector_PinSocket_2.54mm:PinSocket_2x04_P2.54mm_Vertical
- removed R18: 300, Custom:R_0603_HandSolder_ValuePrinted
- removed R19: 16.2K, Custom:R_0603_HandSolder_ValuePrinted
- added J4: Conn_UART, Connector_PinHeader_2.54mm:PinHeader_1x04_P2.54mm_Vertical, F.Cu at (123.5, 85.1)
- C1, C2, C3, C6: footprint Custom:C_0603_HandSolder_ValuePrinted -> Capacitor_SMD:C_0603_1608Metric
- C4: value 10nF -> 10uF; footprint Custom:C_0603_HandSolder_ValuePrinted -> Capacitor_SMD:C_0603_1608Metric
- C5: value 10uF -> 10nF; footprint Custom:C_0603_HandSolder_ValuePrinted -> Capacitor_SMD:C_0603_1608Metric
- D1: value PWR_LED -> SMF24A; footprint Diode_SMD:D_0603_1608Metric_Pad1.05x0.95mm_HandSolder -> Diode_SMD:D_SMF
- D3: value SMF24A -> PWR_LED; footprint Diode_SMD:D_SMF -> Diode_SMD:D_0603_1608Metric
- J1: value Conn_VCC_Alt -> Conn_VCC; footprint TerminalBlock_Phoenix:TerminalBlock_Phoenix_MKDS-1,5-2_1x02_P5.00mm_Horizontal -> Custom:BarrelJack_GCT_DCJ200-10-A_Horizontal
- J2: value Conn_VCC -> Conn_LED; footprint Custom:BarrelJack_GCT_DCJ200-10-A_Horizontal -> footprints:CON_532540670_MOL
- J3: value Conn_LED -> Conn_Aux; footprint footprints:CON_532540670_MOL -> Connector_PinSocket_2.54mm:PinSocket_2x04_P2.54mm_Vertical
- L1: footprint Inductor_SMD:L_1210_3225Metric_Pad1.42x2.65mm_HandSolder -> Inductor_SMD:L_1210_3225Metric
- Q1, Q2, Q3, Q4, Q5: footprint Package_TO_SOT_SMD:SOT-23 -> Custom:SOT-23
- R1, R10, R11, R12, R13, R2, R3, R4, R5, R6, R7, R8, R9: footprint Custom:R_0603_HandSolder_ValuePrinted -> Resistor_SMD:R_0603_1608Metric
- R14: value 0 -> 100K; footprint Resistor_SMD:R_0603_1608Metric_Pad0.98x0.95mm_HandSolder -> Resistor_SMD:R_0603_1608Metric
- R15: value 0 -> 49.9K; footprint Resistor_SMD:R_0603_1608Metric_Pad0.98x0.95mm_HandSolder -> Resistor_SMD:R_0603_1608Metric
- R16: value 100K -> 16.2K; footprint Custom:R_0603_HandSolder_ValuePrinted -> Resistor_SMD:R_0603_1608Metric
- R17: value 49.9K -> 300; footprint Custom:R_0603_HandSolder_ValuePrinted -> Resistor_SMD:R_0603_1608Metric
- moved JP1 46.5 mm to (105.1, 74.0), turned to -90 degrees
- moved R13 37.3 mm to (110.0, 74.7)
- moved U1 37.0 mm to (108.9, 82.8), turned to 180 degrees
- moved SW1 35.7 mm to (99.5, 83.1), turned to 90 degrees
- moved Q5 33.7 mm to (134.8, 59.1), turned to 0 degrees
- moved C2 33.5 mm to (99.6, 79.6), turned to 180 degrees
- moved R11 32.7 mm to (99.6, 77.8), turned to 180 degrees
- moved JP2 32.7 mm to (122.6, 81.9)
- moved R14 32.2 mm to (120.2, 69.4)
- moved J2 31.9 mm to (140.1, 80.1), turned to 90 degrees
- moved R15 29.1 mm to (124.8, 72.4), turned to -90 degrees
- moved R10 28.8 mm to (130.6, 58.1)
- moved C1 28.2 mm to (118.5, 87.0), turned to 180 degrees
- moved Q4 25.8 mm to (134.8, 64.1), turned to 0 degrees
- moved C3 25.8 mm to (118.5, 85.2), turned to 180 degrees
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Connections:
- C4 pad 1: Net-(U2-BST) -> VCC
- C4 pad 2: Net-(D2-K) -> GND
- C5 pad 1: VCC -> Net-(U2-BST)
- C5 pad 2: GND -> Net-(D2-K)
- D1 pad 1: +3.3V -> VCC
- D1 pad 2: Net-(D1-A) -> GND
- D3 pad 1: VCC -> +3.3V
- D3 pad 2: GND -> Net-(D3-A)
- F1 pad 2: Net-(J1-Pin_2) -> Net-(F1-Pad2)
- J1 pad 1: GND -> Net-(F1-Pad2)
- J1 pad 2: Net-(J1-Pin_2) -> GND
- J2 pad 1: Net-(J1-Pin_2) -> VCC
- J2 pad 2: GND -> /W
- J2 pad 3: unconnected-(J2-Pad3) -> /B
- J3 pad 1: VCC -> GND
- J3 pad 2: /W -> +3.3V
- J3 pad 3: /B -> /IO0
- J3 pad 4: /R -> /IO1
- J3 pad 5: /G -> /IO2
- J3 pad 6: /WW -> /IO3
- R14 pad 1: /RX -> Net-(U2-EN)
- R14 pad 2: Net-(J5-Pin_3) -> VCC
- R15 pad 1: /TX -> Net-(U2-FB)
- R15 pad 2: Net-(J5-Pin_2) -> +3.3V
- R16 pad 1: Net-(U2-EN) -> GND
- R16 pad 2: VCC -> Net-(U2-FB)
- R17 pad 1: Net-(U2-FB) -> GND
- R17 pad 2: +3.3V -> Net-(D3-A)
Routing:
- net +3.3V: track 114.4 -> 15.2 mm
- net /PWM_W: track 10.7 -> 42.4 mm, vias 0 -> 4
- net /TX: track 5.44 -> 31.6 mm, vias 0 -> 1
- net VCC: track 77.4 -> 51.6 mm
- net /WW: track 38.2 -> 12.8 mm, vias 1 -> 0
- net /PWM_B: track 14.4 -> 36.0 mm, vias 0 -> 2
- net /G: track 30.9 -> 9.77 mm, vias 1 -> 0
- net /IO3: track 47.8 -> 26.9 mm
- net /RX: track 7.43 -> 28.3 mm, vias 0 -> 1
- net Net-(J1-Pin_2): track 19.9 -> 0.00 mm
- net /IO2: track 45.7 -> 28.8 mm
- net /IO0: track 51.8 -> 35.7 mm
- net /R: track 23.6 -> 7.85 mm, vias 1 -> 0
- net Net-(U1-EN): track 7.54 -> 19.6 mm, vias 0 -> 2
- net /PWM_R: track 19.9 -> 31.2 mm, vias 0 -> 4
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- added copper zone on F.Cu, net +3.3V
- added copper zone on B.Cu, net GND
- added copper zone on F.Cu, net Net-(F1-Pad2)
- added copper zone on F.Cu, net VCC
Other:
- board size 60 x 40 mm -> 50 x 40 mm
- board text removed: "PWR W B R G WW"

Commit message: 2024-06-04 002
Parts:
- removed the J1 at (108.7, 64.3)
- added J1: Conn_VCC, TerminalBlock_Phoenix:TerminalBlock_Phoenix_MKDS-1,5-2_1x02_P5.00mm_Horizontal, F.Cu at (113.9, 57.7)
- added J1: Conn_VCC, TerminalBlock_Phoenix:TerminalBlock_Phoenix_MKDS-1,5-2_1x02_P5.00mm_Horizontal, F.Cu at (100.0, 63.6)
- added J5: PWR_AUX, Connector_PinHeader_2.54mm:PinHeader_1x03_P2.54mm_Vertical, F.Cu at (135.3, 83.6)
- added JP3: SolderJumper_2_Open, Jumper:SolderJumper-2_P1.3mm_Open_RoundedPad1.0x1.5mm, F.Cu at (115.2, 78.0)
- added TP1: PWM_W, TestPoint:TestPoint_Loop_D2.50mm_Drill1.0mm, F.Cu at (141.8, 94.6)
- added TP2: PWM_B, TestPoint:TestPoint_Loop_D2.50mm_Drill1.0mm, F.Cu at (141.8, 87.6)
- added TP3: PWM_R, TestPoint:TestPoint_Loop_D2.50mm_Drill1.0mm, F.Cu at (136.8, 77.6)
- added TP4: PWM_G, TestPoint:TestPoint_Loop_D2.50mm_Drill1.0mm, F.Cu at (136.8, 70.6)
- added TP5: PWM_WW, TestPoint:TestPoint_Loop_D2.50mm_Drill1.0mm, F.Cu at (136.8, 63.6)
- D2: value B230A -> B230-13-F; footprint Diode_SMD:D_SMA -> Diode_SMD:D_SMB
- J4: footprint Connector_PinHeader_2.54mm:PinHeader_1x04_P2.54mm_Vertical -> Connector_PinHeader_2.00mm:PinHeader_1x04_P2.00mm_Vertical
- JP1: value Boot_Mode -> Boot Mode 1
- JP2: value SolderJumper_2_Open -> Boot Mode 2; footprint Jumper:SolderJumper-2_P1.3mm_Open_RoundedPad1.0x1.5mm -> Connector_PinHeader_2.00mm:PinHeader_1x03_P2.00mm_Vertical
- R13: value 100K -> 4.7K
- moved D3 32.7 mm to (126.1, 92.3)
- moved R17 29.5 mm to (124.1, 92.3)
- moved R13 24.0 mm to (121.5, 95.8)
- moved JP1 23.6 mm to (121.5, 91.1), turned to 0 degrees
- moved R2 23.0 mm to (145.7, 95.6)
- moved R4 21.6 mm to (145.7, 88.6)
- moved Q1 21.4 mm to (149.6, 94.5)
- moved R1 20.2 mm to (145.7, 93.6)
- moved Q2 20.0 mm to (149.6, 87.5)
- moved C2 19.4 mm to (115.1, 91.3), turned to -90 degrees
- moved R3 18.9 mm to (145.7, 86.6)
- moved J4 18.7 mm to (109.2, 73.1)
- moved SW1 18.3 mm to (113.4, 94.9), turned to 0 degrees
- moved R11 17.4 mm to (109.5, 92.1), turned to 90 degrees
- moved C1 15.9 mm to (103.4, 92.1), turned to 90 degrees
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Connections:
- JP2 pad 1: +3.3V -> /PWM_WW
- JP2 pad 2: Net-(J4-Pin_1) -> Net-(JP2-C)
- R13 pad 2: /PWM_WW -> Net-(JP2-B)
- U1 pad 10: unconnected-(U1-NC_4-Pad10) -> (no net)
- U1 pad 15: unconnected-(U1-NC_5-Pad15) -> (no net)
- U1 pad 17: unconnected-(U1-NC_6-Pad17) -> (no net)
- U1 pad 22: /PWM_WW -> Net-(JP2-C)
- U1 pad 24: unconnected-(U1-NC_7-Pad24) -> (no net)
- U1 pad 25: unconnected-(U1-NC_8-Pad25) -> (no net)
- U1 pad 28: unconnected-(U1-NC_9-Pad28) -> (no net)
- U1 pad 29: unconnected-(U1-NC_10-Pad29) -> (no net)
- U1 pad 32: unconnected-(U1-NC_11-Pad32) -> (no net)
- U1 pad 33: unconnected-(U1-NC_12-Pad33) -> (no net)
- U1 pad 34: unconnected-(U1-NC_13-Pad34) -> (no net)
- U1 pad 35: unconnected-(U1-NC_14-Pad35) -> (no net)
- U1 pad 4: unconnected-(U1-NC_1-Pad4) -> (no net)
- U1 pad 7: unconnected-(U1-NC_2-Pad7) -> (no net)
- U1 pad 9: unconnected-(U1-NC_3-Pad9) -> (no net)
Routing:
- net GND: track 57.0 -> 0.00 mm, vias 34 -> 0
- net VCC: track 51.6 -> 5.09 mm, vias 0 -> 5
- net Net-(JP2-C): track 0.00 -> 22.9 mm, vias 0 -> 1
- net /IO9: track 3.96 -> 26.8 mm, vias 0 -> 1
- net /TX: track 31.6 -> 12.9 mm, vias 1 -> 0
- net /RX: track 28.3 -> 9.76 mm, vias 1 -> 0
- net /IO0: track 35.7 -> 22.1 mm, vias 1 -> 3
- net /W: track 4.83 -> 18.4 mm
- net /IO1: track 41.3 -> 27.9 mm, vias 1 -> 3
- net /PWM_WW: track 35.8 -> 48.8 mm, vias 2 -> 1
- net /IO2: track 28.8 -> 41.7 mm, vias 1 -> 0
- net /PWM_R: track 31.2 -> 43.3 mm, vias 4 -> 1
- net +3.3V: track 15.2 -> 7.06 mm, vias 2 -> 10
- net /PWM_G: track 30.8 -> 38.5 mm, vias 4 -> 1
- net Net-(U1-EN): track 19.6 -> 11.9 mm, vias 2 -> 0
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- added copper zone on B.Cu, net +3.3V
- added copper zone on B.Cu, net Net-(J1-Pin_2)
- added copper zone on B.Cu, net VCC
- removed copper zone on B.Cu, net GND
Other:
- board size 50 x 40 mm -> 65 x 45 mm

Commit message: 2024-06-05
Parts:
- D3: footprint Diode_SMD:D_0603_1608Metric -> Diode_SMD:D_0603_1608Metric_Pad1.05x0.95mm_HandSolder
- F1: value 24VDC 10A -> 24VDC 5A
- R17: footprint Resistor_SMD:R_0603_1608Metric -> Resistor_SMD:R_0603_1608Metric_Pad0.98x0.95mm_HandSolder
- moved C4 4.20 mm to (123.1, 69.5)
- moved C5 4.20 mm to (130.5, 73.8)
- moved D2 4.20 mm to (120.9, 73.2)
- moved L1 4.20 mm to (126.8, 75.0)
- moved R15 4.20 mm to (130.5, 70.3)
- moved R16 4.20 mm to (130.5, 66.8)
- moved U2 4.20 mm to (127.3, 70.5)
- moved R14 4.20 mm to (125.5, 67.4)
- moved C6 4.20 mm to (123.9, 77.6)
- moved J5 2.00 mm to (135.3, 81.6)
Routing:
- net /IO0: track 22.1 -> 25.9 mm
- net /PWM_R: track 43.3 -> 40.3 mm
- net /PWM_W: track 42.2 -> 45.2 mm
- net /PWM_G: track 38.5 -> 35.9 mm
- net /PWM_WW: track 48.8 -> 46.5 mm
- net /IO1: track 27.9 -> 29.1 mm
- net /PWM_B: track 38.9 -> 40.0 mm
- net Net-(JP2-C): track 22.9 -> 23.7 mm
- net /IO2: track 41.7 -> 41.0 mm
- net Net-(J4-Pin_1): track 8.91 -> 8.33 mm
Other:
- outline, holes or cut-outs redrawn
- board text added: "+24V"
- board text added: "+24V (fused)"
- board text added: "+24V (no fuse)"
- board text added: "+3V3"
- board text added: "2024-06-05"
- board text added: "24V|W|B|R|G|WW"
- board text added: "3V3? RX TX GND"
- board text added: "3V3|GND|24V"
- board text added: "<CodedSakura/>"
- board text added: "=4mm =65mm =55mm =45mm =35mm"
- board text added: "B"
- board text added: "G"
- board text added: "GND"
- board text added: "GND 3V3"
- board text added: "JLCJLCJLCJLC"
- board text added: "LED Driver"
- board text added: "PWR"
- board text added: "R"
- board text added: "RESET"
- board text added: "REV: 1.0"
- board text added: "RGB-CCW LED 24V@3A MAX"
- board text added: "UP|IO8|WW"
- board text added: "UP|IO9"
- board text added: "W"
- board text added: "WW"
- board text added: "h"
- board text added: "w"
- board text added: "w x h y"
- board text added: "x"
- board text added: "y"
- board text added: "|0|2|18 |1|3|19"

Commit message: 2024-11-23
Parts:
- removed JP3: SolderJumper_2_Open, Jumper:SolderJumper-2_P1.3mm_Open_RoundedPad1.0x1.5mm
- J4: footprint Connector_PinHeader_2.00mm:PinHeader_1x04_P2.00mm_Vertical -> Connector_PinHeader_2.54mm:PinHeader_1x04_P2.54mm_Vertical
- JP1: footprint Connector_PinHeader_2.00mm:PinHeader_1x02_P2.00mm_Vertical -> Connector_PinHeader_2.54mm:PinHeader_1x02_P2.54mm_Vertical
- JP2: footprint Connector_PinHeader_2.00mm:PinHeader_1x03_P2.00mm_Vertical -> Connector_PinHeader_2.54mm:PinHeader_1x03_P2.54mm_Vertical
- moved J4 7.45 mm to (115.4, 77.3), turned to 180 degrees
- moved JP1 1.00 mm to (121.5, 90.1)
- moved JP2 1.00 mm to (117.9, 90.1)
Connections:
- J4 pad 1: Net-(J4-Pin_1) -> +3.3V
- J4 pad 2: /RX -> GND
- J4 pad 3: /TX -> /RX
- J4 pad 4: GND -> /TX
Routing:
- net Net-(J4-Pin_1): track 8.33 -> 0.00 mm
- net /IO0: track 25.9 -> 22.3 mm
- net /PWM_B: track 40.0 -> 36.8 mm
- net /IO1: track 29.1 -> 26.8 mm
- net /RX: track 9.76 -> 11.1 mm
- net /PWM_WW: track 46.5 -> 45.5 mm
- net /PWM_W: track 45.2 -> 46.1 mm
- net Net-(JP2-C): track 23.7 -> 22.7 mm
- net /IO18: track 36.3 -> 37.0 mm
- net +3.3V: vias 10 -> 9
Other:
- board text added: "2024-09-01"
- board text added: "DOWN|IO9"
- board text added: "GND TX RX 3V3"
- board text added: "REV: 1.1"
- board text removed: "2024-06-05"
- board text removed: "3V3? RX TX GND"
- board text removed: "REV: 1.0"
- board text removed: "UP|IO9"

Commit message: 2024-11-24 (sub-par pcb)
Parts:
- removed the J1 at (113.9, 57.7)
- removed the J1 at (100.0, 63.6)
- removed JP2: Boot Mode 2, Connector_PinHeader_2.54mm:PinHeader_1x03_P2.54mm_Vertical
- removed R13: 4.7K, Resistor_SMD:R_0603_1608Metric
- removed TP1: PWM_W, TestPoint:TestPoint_Loop_D2.50mm_Drill1.0mm
- removed TP2: PWM_B, TestPoint:TestPoint_Loop_D2.50mm_Drill1.0mm
- removed TP3: PWM_R, TestPoint:TestPoint_Loop_D2.50mm_Drill1.0mm
- removed TP4: PWM_G, TestPoint:TestPoint_Loop_D2.50mm_Drill1.0mm
- removed TP5: PWM_WW, TestPoint:TestPoint_Loop_D2.50mm_Drill1.0mm
- added J1: Conn_VCC_screw, TerminalBlock_Phoenix:TerminalBlock_Phoenix_MKDS-1,5-2_1x02_P5.00mm_Horizontal, F.Cu at (105.2, 77.1)
- added J6: Conn_VCC, Connector_JST:JST_VH_B2PS-VH_1x02_P3.96mm_Horizontal, F.Cu at (115.2, 62.5)
- J2: footprint footprints:CON_532540670_MOL -> Connector_JST:JST_VH_B6PS-VH_1x06_P3.96mm_Horizontal
- J4: value Conn_UART -> USB_B_Mini; footprint Connector_PinHeader_2.54mm:PinHeader_1x04_P2.54mm_Vertical -> Connector_USB:USB_Mini-B_AdamTech_MUSB-B5-S-VT-TSMT-1_SMD_Vertical
- JP1: value Boot Mode 1 -> VBUS_to_VCC
- moved SW1 55.1 mm to (156.4, 60.5), turned to 90 degrees
- moved R11 55.0 mm to (157.5, 65.1)
- moved C2 48.0 mm to (155.3, 65.1), turned to 90 degrees
- moved C1 41.7 mm to (135.6, 65.4), turned to 0 degrees
- moved U1 40.3 mm to (144.9, 69.5), turned to 0 degrees
- moved C3 39.1 mm to (135.6, 67.2), turned to 0 degrees
- moved R2 36.7 mm to (163.6, 63.6)
- moved R1 36.6 mm to (163.6, 61.6)
- moved Q1 36.6 mm to (167.4, 62.6)
- moved R12 36.3 mm to (133.0, 66.3), turned to -90 degrees
- moved D3 33.6 mm to (119.7, 59.3), turned to 180 degrees
- moved J4 32.1 mm to (147.3, 80.4), turned to -90 degrees
- moved R17 31.1 mm to (119.7, 61.5), turned to 180 degrees
- moved R4 27.6 mm to (163.6, 67.6)
- moved R3 27.6 mm to (163.6, 65.6)
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Connections:
- J2 pad 2: /W -> /WW
- J2 pad 3: /B -> /G
- J2 pad 5: /G -> /B
- J2 pad 6: /WW -> /W
- J3 pad 3: /IO0 -> /IO3
- J3 pad 4: /IO1 -> /IO2
- J3 pad 5: /IO2 -> /IO20
- J3 pad 6: /IO3 -> /IO21
- J3 pad 7: /IO18 -> /IO1
- J3 pad 8: /IO19 -> /IO0
- J4 pad 1: +3.3V -> Net-(J4-VBUS)
- J4 pad 2: GND -> /USB_D-
- J4 pad 3: /RX -> /USB_D+
- J4 pad 4: /TX -> unconnected-(J4-ID-Pad4)
- JP1 pad 1: /IO9 -> Net-(J4-VBUS)
- JP1 pad 2: GND -> VCC
- U1 pad 18: /PWM_R -> /PWM_WW
- U1 pad 20: /PWM_B -> /PWM_R
- U1 pad 21: /PWM_W -> /PWM_B
- U1 pad 22: Net-(JP2-C) -> /PWM_W
- U1 pad 23: /IO9 -> unconnected-(U1-IO9-Pad23)
- U1 pad 26: /IO18 -> /USB_D-
- U1 pad 27: /IO19 -> /USB_D+
- U1 pad 30: /RX -> /IO20
- U1 pad 31: /TX -> /IO21
Routing:
- net VCC: track 5.19 -> 67.5 mm, vias 5 -> 7
- net GND: track 0.00 -> 48.2 mm, vias 0 -> 23
- net /IO19: track 38.9 -> 0.00 mm, vias 3 -> 0
- net /IO18: track 37.0 -> 0.00 mm, vias 3 -> 0
- net /IO9: track 26.3 -> 0.00 mm, vias 1 -> 0
- net /PWM_WW: track 45.5 -> 19.6 mm, vias 1 -> 0
- net /IO2: track 41.0 -> 15.4 mm
- net /IO3: track 34.5 -> 10.3 mm
- net Net-(JP2-C): track 22.7 -> 0.00 mm, vias 1 -> 0
- net /IO21: track 0.00 -> 22.3 mm, vias 0 -> 1
- net /IO20: track 0.00 -> 19.3 mm, vias 0 -> 1
- net /PWM_W: track 46.1 -> 27.1 mm, vias 3 -> 0
- net Net-(U1-EN): track 11.9 -> 30.1 mm, vias 0 -> 2
- net /IO1: track 26.8 -> 9.28 mm, vias 3 -> 1
- net /PWM_R: track 40.3 -> 23.0 mm, vias 1 -> 0
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- added copper zone on B.Cu, net GND
Other:
- board size 65 x 45 mm -> 90 x 30 mm
- board text removed: "+24V"
- board text removed: "+24V (fused)"
- board text removed: "+24V (no fuse)"
- board text removed: "+3V3"
- board text removed: "2024-09-01"
- board text removed: "24V|W|B|R|G|WW"
- board text removed: "3V3|GND|24V"
- board text removed: "<CodedSakura/>"
- board text removed: "=4mm =65mm =55mm =45mm =35mm"
- board text removed: "B"
- board text removed: "DOWN|IO9"
- board text removed: "G"
- board text removed: "GND"
- board text removed: "GND 3V3"
- board text removed: "GND TX RX 3V3"
- board text removed: "JLCJLCJLCJLC"
- board text removed: "LED Driver"
- board text removed: "PWR"
- board text removed: "R"
- board text removed: "RESET"
- board text removed: "REV: 1.1"
- board text removed: "RGB-CCW LED 24V@3A MAX"
- board text removed: "UP|IO8|WW"
- board text removed: "W"
- board text removed: "WW"
- board text removed: "h"
- board text removed: "w"
- board text removed: "w x h y"
- board text removed: "x"
- board text removed: "y"
- board text removed: "|0|2|18 |1|3|19"

Commit message: 2024-11-24 (better pcb)
Parts:
- moved R1 14.9 mm to (155.4, 74.0), turned to -90 degrees
- moved Q1 13.4 mm to (156.4, 70.2), turned to 90 degrees
- moved R2 12.2 mm to (157.3, 74.0), turned to -90 degrees
- moved J1 0.50 mm to (105.2, 77.6)
- moved C5 0.49 mm to (131.0, 66.5)
- moved C6 0.49 mm to (124.3, 70.3)
- moved D2 0.49 mm to (121.4, 65.9)
- moved R15 0.49 mm to (131.0, 63.0)
- moved R16 0.49 mm to (131.0, 59.5)
- moved R14 0.49 mm to (126.0, 60.2)
- moved U2 0.49 mm to (127.7, 63.2)
- moved C4 0.49 mm to (123.6, 62.3)
- moved L1 0.49 mm to (127.2, 67.7)
- moved R17 0.39 mm to (119.9, 61.2)
- moved D3 0.39 mm to (119.9, 59.0)
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Routing:
- net VCC: track 67.5 -> 7.08 mm, vias 7 -> 10
- net /W: track 6.12 -> 25.6 mm
- net /PWM_W: track 27.1 -> 8.34 mm
- net +3.3V: track 21.6 -> 16.6 mm
- net GND: track 48.2 -> 44.7 mm, vias 23 -> 22
Other:
- outline, holes or cut-outs redrawn
- board text added: "24VDC 5A"
- board text added: "3V3 GND IO2 IO3 IO21 IO20 IO0 IO1"
- board text added: "3V3|GND|VCC"
- board text added: "<CodedSakura/> 2024-11-24"
- board text added: "LED Driver"
- board text added: "PWR"
- board text added: "Power by USB"
- board text added: "RESET"
- board text added: "REV: 2.0"
- board text added: "SMF24A"
